Commit message: update file

File: my_worlds/urdf/leo.urdf.xacro (robot description, xacro)
@@ -2,5 +2,5 @@
 <robot xmlns:xacro="http://www.ros.org/wiki/xacro"
        name="leo">
-  <xacro:include filename="$(find leo_description)/urdf/macros.xacro"/>
+  <xacro:include filename="$(find my_worlds)/urdf/macros.xacro"/>
   <xacro:leo/>
 </robot>

File: my_worlds/urdf/leo_sim.urdf.xacro (robot description, xacro)
@@ -4,5 +4,5 @@
   <xacro:arg name="fixed" default="false"/>
   <xacro:arg name="robot_ns" default=""/>
-  <xacro:include filename="$(find leo_description)/urdf/macros.xacro"/>
+  <xacro:include filename="$(find my_worlds)/urdf/macros.xacro"/>
   <xacro:leo_sim robot_ns="$(arg robot_ns)"
                  fixed="$(arg fixed)"/>

File: my_worlds/urdf/macros.xacro (robot description, xacro)
@@ -19,10 +19,10 @@
         <visual>
           <geometry>
-            <mesh filename="package://leo_description/models/Rocker.dae"/>
+            <mesh filename="package://my_worlds/models/Rocker.dae"/>
           </geometry>
         </visual>
         <collision>
           <geometry>
-            <mesh filename="package://leo_description/models/Rocker_outline.stl"/>
+            <mesh filename="package://my_worlds/models/Rocker_outline.stl"/>
           </geometry>
         </collision>
@@ -41,5 +41,5 @@
         <visual>
           <geometry>
-            <mesh filename="package://leo_description/models/Wheel${model}.dae"/>
+            <mesh filename="package://my_worlds/models/Wheel${model}.dae"/>
           </geometry>
         </visual>
@@ -58,5 +58,5 @@
         <collision>
           <geometry>
-            <mesh filename="package://leo_description/models/Wheel_outline.stl"/>
+            <mesh filename="package://my_worlds/models/Wheel_outline.stl"/>
           </geometry>
         </collision>
@@ -78,10 +78,10 @@
       <visual>
         <geometry>
-          <mesh filename="package://leo_description/models/Chassis.dae"/>
+          <mesh filename="package://my_worlds/models/Chassis.dae"/>
         </geometry>
       </visual>
       <collision>
         <geometry>
-          <mesh filename="package://leo_description/models/Chassis_outline.stl"/>
+          <mesh filename="package://my_worlds/models/Chassis_outline.stl"/>
         </geometry>
       </collision>
@@ -105,5 +105,5 @@
         <visual>
           <geometry>
-            <mesh filename="package://leo_description/models/Antenna.dae"/>
+            <mesh filename="package://my_worlds/models/Antenna.dae"/>
           </geometry>
         </visual>
