Commit message: update file

File: my_worlds/urdf/car.urdf.xacro (robot description, xacro)
@@ -1,6 +1,6 @@
 <?xml version="1.0" encoding="utf-8"?>
 <robot xmlns:xacro="http://www.ros.org/wiki/xacro"
-       name="leo">
+       name="mycar">
   <xacro:include filename="$(find my_worlds)/urdf/macros.xacro"/>
-  <xacro:leo/>
+  <xacro:mycar/>
 </robot>

File: my_worlds/urdf/car_sim.urdf.xacro (robot description, xacro)
@@ -1,9 +1,9 @@
 <?xml version="1.0"?>
 <robot xmlns:xacro="http://ros.org/wiki/xacro"
-       name="leo_sim">
+       name="car_sim">
   <xacro:arg name="fixed" default="false"/>
   <xacro:arg name="robot_ns" default=""/>
   <xacro:include filename="$(find my_worlds)/urdf/macros.xacro"/>
-  <xacro:leo_sim robot_ns="$(arg robot_ns)"
+  <xacro:car_sim robot_ns="$(arg robot_ns)"
                  fixed="$(arg fixed)"/>
 </robot>

File: my_worlds/urdf/macros.xacro (robot description, xacro)
@@ -1,5 +1,5 @@
 <?xml version="1.0" encoding="utf-8"?>
 <robot xmlns:xacro="http://www.ros.org/wiki/xacro">
-  <xacro:macro name="leo"
+  <xacro:macro name="mycar"
                params="default_antenna:=true
                        rockers_fixed:=true
@@ -199,6 +199,6 @@
     </joint>
   </xacro:macro>
-  <!-- LEO GAZEBO -->
-  <xacro:macro name="leo_gazebo"
+  <!-- GAZEBO -->
+  <xacro:macro name="my_worlds"
                params="robot_ns:=''">
     <xacro:property name="link_prefix" value=""/>
@@ -365,5 +365,5 @@
     </transmission>
   </xacro:macro>
-  <xacro:macro name="leo_sim"
+  <xacro:macro name="car_sim"
                params="default_antenna:=true
                        fixed:=false
@@ -373,8 +373,8 @@
       <xacro:property name="link_prefix" value="${robot_ns}/"/>
     </xacro:if>
-    <xacro:leo default_antenna="${default_antenna}"
+    <xacro:mycar default_antenna="${default_antenna}"
                rockers_fixed="false"
                link_prefix="${link_prefix}"/>
-    <xacro:leo_gazebo robot_ns="${robot_ns}"/>
+    <xacro:my_worlds robot_ns="${robot_ns}"/>
     <xacro:if value="${fixed}">
       <link name="world"/>
